Commit message: Fix broken xacro

File: leo_rover_description/urdf/leo_gazebo.xacro (robot description, xacro)
@@ -139,5 +139,5 @@
         <robot_param>robot_description</robot_param>
         <robot_param_node>robot_state_publisher</robot_param_node>
-        <parameters>/home/marco/simulations_ros2_devel/src/leo_simulator/leo_rover_description/config/controllers.yaml</parameters>
+        <parameters>$(find leo_rover_description)/config/controllers.yaml</parameters>
     </plugin>
     </gazebo>

File: leo_rover_description/urdf/leo_rover.urdf.xacro (robot description, xacro)
@@ -300,4 +300,5 @@
       <child link="imu_frame"/>
     </joint>
+    <link name="imu_frame"/>
   <!-- LEO GAZEBO -->
     <gazebo>
@@ -435,5 +436,5 @@
         <robot_param>robot_description</robot_param>
         <robot_param_node>robot_state_publisher</robot_param_node>
-        <parameters>/home/marco/leo_rover_ws/ros2_packages/src/leo_simulator/leo_rover_description/config/controllers.yaml</parameters>
+        <parameters>$(find leo_rover_description)/config/controllers.yaml</parameters>
       </plugin>
     </gazebo>
