Commit message: Update

File: leo_rover_description/urdf/leo_rover.urdf.xacro (robot description, xacro)
@@ -21,10 +21,10 @@
       <visual>
         <geometry>
-          <mesh filename="model://Chassis.dae"/>
-        </geometry>
-      </visual>
-      <collision>
-        <geometry>
-          <mesh filename="model://Chassis_outline.stl"/>
+          <mesh filename="file://$(find leo_rover_description)/models/Chassis.dae"/>
+        </geometry>
+      </visual>
+      <collision>
+        <geometry>
+          <mesh filename="file://$(find leo_rover_description)/models/Chassis_outline.stl"/>
         </geometry>
       </collision>
@@ -50,10 +50,10 @@
       <visual>
         <geometry>
-          <mesh filename="model://Rocker.dae"/>
-        </geometry>
-      </visual>
-      <collision>
-        <geometry>
-          <mesh filename="model://Rocker_outline.stl"/>
+          <mesh filename="file://$(find leo_rover_description)/models/Rocker.dae"/>
+        </geometry>
+      </visual>
+      <collision>
+        <geometry>
+          <mesh filename="file://$(find leo_rover_description)/models/Rocker_outline.stl"/>
         </geometry>
       </collision>
@@ -80,10 +80,10 @@
       <visual>
         <geometry>
-          <mesh filename="model://Rocker.dae"/>
-        </geometry>
-      </visual>
-      <collision>
-        <geometry>
-          <mesh filename="model://Rocker_outline.stl"/>
+          <mesh filename="file://$(find leo_rover_description)/models/Rocker.dae"/>
+        </geometry>
+      </visual>
+      <collision>
+        <geometry>
+          <mesh filename="file://$(find leo_rover_description)/models/Rocker_outline.stl"/>
         </geometry>
       </collision>
@@ -109,5 +109,5 @@
       <visual>
         <geometry>
-          <mesh filename="model://WheelA.dae"/>
+          <mesh filename="file://$(find leo_rover_description)/models/WheelA.dae"/>
         </geometry>
       </visual>
@@ -126,5 +126,5 @@
       <collision>
         <geometry>
-          <mesh filename="model://Wheel_outline.stl"/>
+          <mesh filename="file://$(find leo_rover_description)/models/WheelA.stl"/>
         </geometry>
       </collision>
@@ -150,5 +150,5 @@
       <visual>
         <geometry>
-          <mesh filename="model://WheelA.dae"/>
+          <mesh filename="file://$(find leo_rover_description)/models/WheelA.dae"/>
         </geometry>
       </visual>
@@ -167,5 +167,5 @@
       <collision>
         <geometry>
-          <mesh filename="model://Wheel_outline.stl"/>
+          <mesh filename="file://$(find leo_rover_description)/models/WheelA.stl"/>
         </geometry>
       </collision>
@@ -191,5 +191,5 @@
       <visual>
         <geometry>
-          <mesh filename="model://WheelB.dae"/>
+          <mesh filename="file://$(find leo_rover_description)/models/WheelB.dae"/>
         </geometry>
       </visual>
@@ -208,5 +208,5 @@
       <collision>
         <geometry>
-          <mesh filename="model://Wheel_outline.stl"/>
+          <mesh filename="file://$(find leo_rover_description)/models/WheelB.stl"/>
         </geometry>
       </collision>
@@ -232,5 +232,5 @@
       <visual>
         <geometry>
-          <mesh filename="model://WheelB.dae"/>
+          <mesh filename="file://$(find leo_rover_description)/models/WheelB.dae"/>
         </geometry>
       </visual>
@@ -249,8 +249,11 @@
       <collision>
         <geometry>
-          <mesh filename="model://Wheel_outline.stl"/>
-        </geometry>
-      </collision>
-    </link>
+          <mesh filename="file://$(find leo_rover_description)/models/WheelB.stl"/>
+        </geometry>
+      </collision>
+    </link>
+    <link name="camera_frame"/>
+    <link name="camera_optical_frame"/>
+    <link name="imu_frame"/>
     <!-- Antenna link -->
     <joint name="antenna_joint" type="fixed">
@@ -270,5 +273,5 @@
       <visual>
         <geometry>
-          <mesh filename="model://Antenna.dae"/>
+          <mesh filename="file://$(find leo_rover_description)/models/Antenna.dae"/>
         </geometry>
       </visual>
@@ -286,5 +289,4 @@
       <child link="camera_frame"/>
     </joint>
-    <link name="camera_frame"/>
     <!-- Camera optical link -->
     <joint name="camera_optical_joint" type="fixed">
@@ -293,5 +295,4 @@
       <child link="camera_optical_frame"/>
     </joint>
-    <link name="camera_optical_frame"/>
     <!-- Imu link -->
     <joint name="imu_joint" type="fixed">
@@ -300,6 +301,68 @@
       <child link="imu_frame"/>
     </joint>
-    <link name="imu_frame"/>
   <!-- LEO GAZEBO -->
+      <!-- base ODE properties -->
+    <gazebo reference="base_footprint">
+      <kp>1e6</kp>
+      <kd>1.0</kd>
+      <mu1>0.3</mu1>
+      <mu2>0.3</mu2>
+      <minDepth>0.003</minDepth>
+    </gazebo>
+    <gazebo reference="base_link">
+      <kp>1e6</kp>
+      <kd>1.0</kd>
+      <mu1>0.3</mu1>
+      <mu2>0.3</mu2>
+      <minDepth>0.003</minDepth>
+    </gazebo>
+    <!-- rocker ODE properties -->
+    <gazebo reference="rocker_L_link">
+      <kp>1e6</kp>
+      <kd>1.0</kd>
+      <mu1>0.3</mu1>
+      <mu2>0.3</mu2>
+      <minDepth>0.003</minDepth>
+    </gazebo>
+    <gazebo reference="rocker_R_link">
+      <kp>1e6</kp>
+      <kd>1.0</kd>
+      <mu1>0.3</mu1>
+      <mu2>0.3</mu2>
+      <minDepth>0.003</minDepth>
+    </gazebo>
+    <!-- wheel ODE properties -->
+    <gazebo reference="wheel_FL_link">
+      <kp>1e6</kp>
+      <kd>100.0</kd>
+      <mu1>3.0</mu1>
+      <mu2>0.1</mu2>
+      <fdir1>1 0 0</fdir1>
+      <minDepth>0.003</minDepth>
+    </gazebo>
+    <gazebo reference="wheel_FR_link">
+      <kp>1e6</kp>
+      <kd>100.0</kd>
+      <mu1>3.0</mu1>
+      <mu2>0.1</mu2>
+      <fdir1>1 0 0</fdir1>
+      <minDepth>0.003</minDepth>
+    </gazebo>
+    <gazebo reference="wheel_RL_link">
+      <kp>1e6</kp>
+      <kd>100.0</kd>
+      <mu1>3.0</mu1>
+      <mu2>0.1</mu2>
+      <fdir1>1 0 0</fdir1>
+      <minDepth>0.003</minDepth>
+    </gazebo>
+    <gazebo reference="wheel_RR_link">
+      <kp>1e6</kp>
+      <kd>100.0</kd>
+      <mu1>3.0</mu1>
+      <mu2>0.1</mu2>
+      <fdir1>1 0 0</fdir1>
+      <minDepth>0.003</minDepth>
+    </gazebo>
     <gazebo>
       <plugin name="mimic_joint" filename="libmimic_joint_plugin.so">
@@ -364,6 +427,6 @@
         <right_joint>wheel_FR_joint</right_joint>
         <!-- kinematics -->
-        <wheel_separation>0.33</wheel_separation>
-        <wheel_diameter>0.125</wheel_diameter>
+        <wheel_separation>0.355</wheel_separation>
+        <wheel_diameter>0.115</wheel_diameter>
         <!-- output -->
         <publish_odom>true</publish_odom>
